Commit message: v2.2

File: test_ws/src/test_description/urdf/test.urdf.xacro (robot description, xacro)
@@ -2,23 +2,24 @@
 <robot xmlns:xacro="http://www.ros.org/wiki/xacro" name="test_robot">
     <xacro:include filename="$(find test_description)/urdf/test_control.xacro"/>
+    <link name="world"/>
     <link name="base_link">
         <inertial>
-            <origin xyz="0.0 0.0 0.0" rpy="0.0 0.0 0.0"/>
-            <mass value="0.41542"/>
+            <origin xyz="0.00039768 8.0247E-10 0.012605" rpy="0 0 0" />
+            <mass value="0.41542" />
             <inertia ixx="0.00054632" ixy="-4.5067E-09" ixz="5.9528E-07" iyy="0.00053741" iyz="-3.5275E-10" izz="0.0010336" />
         </inertial>
         <visual>
-            <origin xyz="0.0 0.0 0.0" rpy="0.0 0.0 0.0"/>
-            <geometry>
-                <mesh filename="package://test_description/meshes/base_link.STL" scale="1.0 1.0 1.0"/>
-            </geometry>
-            <material name="">
-                <color rgba="0.89412 0.91373 0.92941 1"/>
-            </material>
-        </visual>
-        <collision>
-            <origin xyz="0.0 0.0 0.0" rpy="0.0 0.0 0.0"/>
-            <geometry>
-                <mesh filename="package://test_description/meshes/base_link.STL" scale="1.0 1.0 1.0"/>
+            <origin xyz="0 0 0" rpy="0 0 0" />
+            <geometry>
+                <mesh filename="package://test_description/meshes/base_link.STL" />
+            </geometry>
+            <material name="">
+                <color rgba="0.89412 0.91373 0.92941 1" />
+            </material>
+        </visual>
+        <collision>
+            <origin xyz="0 0 0" rpy="0 0 0" />
+            <geometry>
+                <mesh filename="package://test_description/meshes/base_link.STL" />
             </geometry>
         </collision>
@@ -26,31 +27,192 @@
     <link name="link1">
         <inertial>
-            <origin xyz="0.0 0.0 0.0" rpy="0.0 0.0 0.0"/>
-            <mass value="1.7827"/>
+            <origin xyz="3.9336E-06 -0.0082614 0.0028405" rpy="0 0 0" />
+            <mass value="1.7827" />
             <inertia ixx="0.0031691" ixy="-1.2175E-07" ixz="-2.8349E-08" iyy="0.0029334" iyz="0.00037927" izz="0.0035086" />
         </inertial>
         <visual>
-            <origin xyz="0.0 0.0 0.0" rpy="0.0 0.0 0.0"/>
-            <geometry>
-                <mesh filename="package://test_description/meshes/link1.STL" scale="1.0 1.0 1.0"/>
-            </geometry>
-            <material name="">
-                <color rgba="1.0 1.0 1.0 1.0"/>
-            </material>
-        </visual>
-        <collision>
-            <origin xyz="0.0 0.0 0.0" rpy="0.0 0.0 0.0"/>
-            <geometry>
-                <mesh filename="package://test_description/meshes/link1.STL" scale="1.0 1.0 1.0"/>
-            </geometry>
-        </collision>
-    </link>
+            <origin xyz="0 0 0" rpy="0 0 0" />
+            <geometry>
+                <mesh filename="package://test_description/meshes/link1.STL" />
+            </geometry>
+            <material name="">
+                <color rgba="1 1 1 1" />
+            </material>
+        </visual>
+        <collision>
+            <origin xyz="0 0 0" rpy="0 0 0" />
+            <geometry>
+                <mesh filename="package://test_description/meshes/link1.STL" />
+            </geometry>
+        </collision>
+    </link>
+    <link name="link2">
+        <inertial>
+            <origin xyz="-2.17E-06 0.17637 0.13932" rpy="0 0 0" />
+            <mass value="4.8843" />
+            <inertia ixx="0.022101" ixy="-1.0832E-07" ixz="-1.2727E-07" iyy="0.0066105" iyz="-0.00021178" izz="0.022526" />
+        </inertial>
+        <visual>
+            <origin xyz="0 0 0" rpy="0 0 0" />
+            <geometry>
+                <mesh filename="package://test_description/meshes/link2.STL" />
+            </geometry>
+            <material name="">
+                <color rgba="1 1 1 1" />
+            </material>
+        </visual>
+        <collision>
+            <origin xyz="0 0 0" rpy="0 0 0" />
+            <geometry>
+                <mesh filename="package://test_description/meshes/link2.STL" />
+            </geometry>
+        </collision>
+    </link>
+    <link name="link3">
+        <inertial>
+            <origin xyz="0.20069 -7.9845E-06 0.028008" rpy="0 0 0" />
+            <mass value="2.1495" />
+            <inertia ixx="0.0015747" ixy="-2.8912E-08" ixz="7.3471E-05" iyy="0.0091566" iyz="-1.4815E-07" izz="0.0091573" />
+        </inertial>
+        <visual>
+            <origin xyz="0 0 0" rpy="0 0 0" />
+            <geometry>
+                <mesh filename="package://test_description/meshes/link3.STL" />
+            </geometry>
+            <material name="">
+                <color rgba="1 1 1 1" />
+            </material>
+        </visual>
+        <collision>
+            <origin xyz="0 0 0" rpy="0 0 0" />
+            <geometry>
+                <mesh filename="package://test_description/meshes/link3.STL" />
+            </geometry>
+        </collision>
+    </link>
+    <link name="link4">
+        <inertial>
+            <origin xyz="-5.2274E-07 -0.00070291 -0.006006" rpy="0 0 0" />
+            <mass value="0.53436" />
+            <inertia ixx="0.00041486" ixy="-4.7177E-09" ixz="-1.1841E-09" iyy="0.0004403" iyz="-5.8283E-05" izz="0.00037669" />
+        </inertial>
+        <visual>
+            <origin xyz="0 0 0" rpy="0 0 0" />
+            <geometry>
+                <mesh filename="package://test_description/meshes/link4.STL" />
+            </geometry>
+            <material name="">
+                <color rgba="1 1 1 1" />
+            </material>
+        </visual>
+        <collision>
+            <origin xyz="0 0 0" rpy="0 0 0" />
+            <geometry>
+                <mesh filename="package://test_description/meshes/link4.STL" />
+            </geometry>
+        </collision>
+    </link>
+    <link name="link5">
+        <inertial>
+            <origin xyz="5.2283E-07 0.00070291 -0.006006" rpy="0 0 0" />
+            <mass value="0.53436" />
+            <inertia ixx="0.00041486" ixy="-4.6787E-09" ixz="1.1524E-09" iyy="0.0004403" iyz="5.8283E-05" izz="0.00037669" />
+        </inertial>
+        <visual>
+            <origin xyz="0 0 0" rpy="0 0 0" />
+            <geometry>
+                <mesh filename="package://test_description/meshes/link5.STL" />
+            </geometry>
+            <material name="">
+                <color rgba="1 1 1 1" />
+            </material>
+        </visual>
+        <collision>
+            <origin xyz="0 0 0" rpy="0 0 0" />
+            <geometry>
+                <mesh filename="package://test_description/meshes/link5.STL" />
+            </geometry>
+        </collision>
+    </link>
+    <link name="link6">
+        <inertial>
+            <origin xyz="-1.7556E-08 -0.00045052 -0.021169" rpy="0 0 0" />
+            <mass value="0.16488" />
+            <inertia ixx="7.7869E-05" ixy="-3.3531E-10" ixz="1.915E-10" iyy="7.757E-05" iyz="-7.8331E-08" izz="0.00011744" />
+        </inertial>
+        <visual>
+            <origin xyz="0 0 0" rpy="0 0 0" />
+            <geometry>
+                <mesh filename="package://test_description/meshes/link6.STL" />
+            </geometry>
+            <material name="">
+                <color rgba="0.79216 0.81961 0.93333 1" />
+            </material>
+        </visual>
+        <collision>
+            <origin xyz="0 0 0" rpy="0 0 0" />
+            <geometry>
+                <mesh filename="package://test_description/meshes/link6.STL" />
+            </geometry>
+        </collision>
+    </link>
+    <link name="flan"/>
+    <joint name="world_joint" type="fixed">
+        <origin xyz="0.0 0.0 0.0" rpy="0.0 0.0 0.0"/>
+        <parent link="world"/>
+        <child link="base_link"/>
+    </joint>
     <joint name="joint1" type="revolute">
-        <origin xyz="0.0 0.0 0.096" rpy="0.0 0.0 3.14159"/>
-        <parent link="base_link"/>
-        <child link="link1"/>
-        <axis xyz="0.0 0.0 1.0"/>
-        <limit lower="-3.14159" upper="3.14159" effort="150.0" velocity="2.61993"/>
-        <dynamics damping="0.0" friction="0.0"/>
+        <origin xyz="0 0 0.096" rpy="0 0 3.1416" />
+        <parent link="base_link" />
+        <child link="link1" />
+        <axis xyz="0 0 1" />
+        <limit lower="-6.2832" upper="6.2832" effort="150.0" velocity="2.61993" />
+        <dynamics damping="0" friction="0" />
+    </joint>
+    <joint name="joint2" type="revolute">
+        <origin xyz="0 0 0" rpy="1.5708 -1.5708 0" />
+        <parent link="link1" />
+        <child link="link2" />
+        <axis xyz="0 0 1" />
+        <limit lower="-6.2832" upper="6.2832" effort="150.0" velocity="2.61993" />
+        <dynamics damping="0" friction="0" />
+    </joint>
+    <joint name="joint3" type="revolute">
+        <origin xyz="0 0.418 0" rpy="0 0 1.5708" />
+        <parent link="link2" />
+        <child link="link3" />
+        <axis xyz="0 0 1" />
+        <limit lower="-2.7925" upper="2.7925" effort="150.0" velocity="3.31613" />
+        <dynamics damping="0" friction="0" />
+    </joint>
+    <joint name="joint4" type="revolute">
+        <origin xyz="0.398 0 0.122" rpy="0 0 0" />
+        <parent link="link3" />
+        <child link="link4" />
+        <axis xyz="0 0 1" />
+        <limit lower="-6.2832" upper="6.2832" effort="28.0" velocity="4.53786" />
+        <dynamics damping="0" friction="0" />
+    </joint>
+    <joint name="joint5" type="revolute">
+        <origin xyz="0 0.098 0" rpy="1.5708 0 -3.1416" />
+        <parent link="link4" />
+        <child link="link5" />
+        <axis xyz="0 0 1" />
+        <limit lower="-6.2832" upper="6.2832" effort="28.0" velocity="4.53786" />
+        <dynamics damping="0" friction="0" />
+    </joint>
+    <joint name="joint6" type="revolute">
+        <origin xyz="0 -0.089 0" rpy="-1.5708 0 3.1416" />
+        <parent link="link5" />
+        <child link="link6" />
+        <axis xyz="0 0 1" />
+        <limit lower="-6.2832" upper="6.2832" effort="28.0" velocity="4.53786" />
+        <dynamics damping="0" friction="0" />
+    </joint>
+    <joint name="flan_joint" type="fixed">
+        <origin xyz="0 0 0" rpy="0 0 0" />
+        <parent link="link6" />
+        <child link="flan" />
     </joint>
 </robot>

File: test_ws/src/test_description/urdf/test_control.xacro (robot description, xacro)
@@ -14,6 +14,51 @@
             <state_interface name="effort"/>
         </joint>
+        <joint name="joint2">
+            <command_interface name="position">
+                <param name="min">-3.14</param>
+                <param name="max">3.14</param>
+            </command_interface>
+            <state_interface name="position"/>
+            <state_interface name="velocity"/>
+            <state_interface name="effort"/>
+        </joint>
+        <joint name="joint3">
+            <command_interface name="position">
+                <param name="min">-2.79</param>
+                <param name="max">2.79</param>
+            </command_interface>
+            <state_interface name="position"/>
+            <state_interface name="velocity"/>
+            <state_interface name="effort"/>
+        </joint>
+        <joint name="joint4">
+            <command_interface name="position">
+                <param name="min">-3.14</param>
+                <param name="max">3.14</param>
+            </command_interface>
+            <state_interface name="position"/>
+            <state_interface name="velocity"/>
+            <state_interface name="effort"/>
+        </joint>
+        <joint name="joint5">
+            <command_interface name="position">
+                <param name="min">-3.14</param>
+                <param name="max">3.14</param>
+            </command_interface>
+            <state_interface name="position"/>
+            <state_interface name="velocity"/>
+            <state_interface name="effort"/>
+        </joint>
+        <joint name="joint6">
+            <command_interface name="position">
+                <param name="min">-3.14</param>
+                <param name="max">3.14</param>
+            </command_interface>
+            <state_interface name="position"/>
+            <state_interface name="velocity"/>
+            <state_interface name="effort"/>
+        </joint>
     </ros2_control>
-    <transmission name="tran1">
+    <!-- <transmission name="tran1">
         <type>transmission_interface/SimpleTransmission</type>
         <joint name="joint1">
@@ -23,5 +68,5 @@
             <mechanicalReduction>1.0</mechanicalReduction>
         </actuator>
-    </transmission>
+    </transmission> -->
     <gazebo>
         <plugin filename="libgazebo_ros2_control.so" name="gazebo_ros2_control">
