Commit message: gazebo

File: moveit_ws/src/test_description/urdf/base.xacro (robot description, xacro)
@@ -3,4 +3,5 @@
     <xacro:macro name="base">
         <xacro:property name="PI" value="3.1415926"/>
+        <link name="world" />
         <link name="base_link">
             <visual>
@@ -143,4 +144,9 @@
             </inertial>
         </link>
+        <joint name="world_joint" type="fixed">
+            <parent link="world" />
+            <child link="base_link" />
+            <origin xyz="0 0 0" rpy="0 0 0" />
+        </joint>
         <joint name="joint1" type="revolute">
             <parent link="base_link"/>

File: moveit_ws/src/test_description/urdf/test.urdf.xacro (robot description, xacro)
@@ -3,4 +3,6 @@
     <xacro:include filename="$(find test_description)/urdf/materials.xacro"/>
     <xacro:include filename="$(find test_description)/urdf/base.xacro"/>
+    <xacro:include filename="$(find test_description)/urdf/gazebo.xacro"/>
     <xacro:base/>
+    <xacro:gazebo/>
 </robot>

File: moveit_ws/src/test_moveit_config/config/test_robot.ros2_control.xacro (robot description, xacro)
@@ -5,6 +5,6 @@
         <ros2_control name="${name}" type="system">
             <hardware>
-                <!-- By default, set up controllers for simulation. This won't work on real hardware -->
-                <plugin>mock_components/GenericSystem</plugin>
+                <!-- <plugin>mock_components/GenericSystem</plugin> -->
+                <plugin>gazebo_ros2_control/GazeboSystem</plugin>
             </hardware>
             <joint name="joint1">
